File: hardware/rpi-cm4-base-carrier/rpi-cm4-base-carrier.kicad_pcb (KiCad board)
At the start: 4 copper layers, 169 x 134.1 mm, 81 parts, among them IC1 KTD2052BEVAA-TR, J1 690-019-298-412, J10 Conn_02x05_Odd_Even, J11 XM7B-0442, J2 ERM8-040-01-X-D-EM2-L-XX, J3 USB4105-GF-A, J5 THD-02-R, J6 JT4-1202HL, J7 Micro_SD_Card_Det, J8 Conn_02x10_Odd_Even, J9 690-008-221-904, U1 RT9742SNGV, U2 74LVC1G07SE-7, U4 RT9742GGJ5, U5 FSUSB42MUX, U6 USB2514B-I/M2, U8 AP22653W6, U9 74LVC1G07SE-7, Y1 CX3225CA24000D0HSSCC

Commit message: redundant USBC power schematic created, layout of single USBC input completed@
Parts:
- removed CR1: SMBJ5.0A-TR, footprints:SMBJ5.0A-TR
- removed J3: USB4105-GF-A, USB4105-GF-A:GCT_USB4105-GF-A
- removed R1, R3: 5.1k, Resistor_SMD:R_0603_1608Metric_Pad0.98x0.95mm_HandSolder
- added C27: 100uF, Capacitor_Tantalum_SMD:CP_EIA-7343-31_Kemet-D, F.Cu at (-8.88, 129.2)
- added C28: 1u, RESC2012X140N:RESC2012X140N, F.Cu at (-14.2, 112.9)
- added C29: 1u, RESC2012X140N:RESC2012X140N, F.Cu at (-14.2, 116.0)
- added C30: 1u, RESC2012X140N:RESC2012X140N, F.Cu at (-14.2, 119.0)
- added C31: 10u, Capacitor_SMD:C_0805_2012Metric, F.Cu at (-26.0, 81.2)
- added C32: 1u, RESC2012X140N:RESC2012X140N, F.Cu at (-23.5, 84.5)
- added C33: 1u, RESC2012X140N:RESC2012X140N, F.Cu at (-49.2, 91.5)
- added C34: 1u, RESC2012X140N:RESC2012X140N, F.Cu at (-53.0, 91.3)
- added C35: 1u, RESC2012X140N:RESC2012X140N, F.Cu at (-46.8, 91.5)
- added C36: 10u, Capacitor_SMD:C_0805_2012Metric, F.Cu at (-56.6, 81.2)
- added C37: 1u, RESC2012X140N:RESC2012X140N, F.Cu at (-53.9, 84.8)
- added C38: 100n, Capacitor_SMD:C_0402_1005Metric, F.Cu at (-46.0, 84.8)
- added C39: 1u, RESC2012X140N:RESC2012X140N, F.Cu at (-11.6, 133.7)
- added C40: 1u, RESC2012X140N:RESC2012X140N, F.Cu at (-11.6, 136.7)
- added C41: 100n, Capacitor_SMD:C_0402_1005Metric, F.Cu at (-16.0, 84.8)
- added C42: 1u, RESC2012X140N:RESC2012X140N, F.Cu at (-11.6, 139.8)
- added C43: 1u, RESC2012X140N:RESC2012X140N, F.Cu at (-11.6, 142.8)
- added D12: ESDA25W, SOT65P210X110-3N:SOT65P210X110-3N, F.Cu at (-36.5, 88.4)
- added D13: ESDA25W, SOT65P210X110-3N:SOT65P210X110-3N, F.Cu at (-36.5, 85.4)
- added D14: ESDA25W, SOT65P210X110-3N:SOT65P210X110-3N, F.Cu at (-23.1, 81.3)
- added D16: ESDA25W, SOT65P210X110-3N:SOT65P210X110-3N, F.Cu at (-67.3, 88.7)
- added D17: ESDA25W, SOT65P210X110-3N:SOT65P210X110-3N, F.Cu at (-67.3, 85.7)
- added D18: ESDA25W, SOT65P210X110-3N:SOT65P210X110-3N, F.Cu at (-53.6, 81.3)
- added IC2: LM74610QDGKRQ1, SamacSys_Parts:SOP65P490X110-8N, F.Cu at (-20.9, 128.6)
- added IC3: LM74610QDGKRQ1, SamacSys_Parts:SOP65P490X110-8N, F.Cu at (-20.9, 133.2)
- added J12: USB4105-GF-A, USB4105-GF-A:GCT_USB4105-GF-A, F.Cu at (-64.0, 77.5)
- added J4: USB4105-GF-A, USB4105-GF-A:GCT_USB4105-GF-A, F.Cu at (-33.3, 77.5)
- added MOSFET1: STL11N3LLH6, STL11N3LLH6:POWERFLAT_3P3X3P3_STM, F.Cu at (-21.7, 138.2)
- added MOSFET2: STL11N3LLH6, STL11N3LLH6:POWERFLAT_3P3X3P3_STM, F.Cu at (-21.7, 143.3)
- added Q1: STL6P3LLH6, TRANS_STL6P3LLH6:TRANS_STL6P3LLH6, F.Cu at (-15.7, 81.2)
- added Q2: STL6P3LLH6, TRANS_STL6P3LLH6:TRANS_STL6P3LLH6, F.Cu at (-46.0, 81.2)
- added R2: NF, SamacSys_Parts:RESC1005X40N, F.Cu at (-43.7, 93.8)
- added R22: 22K, SamacSys_Parts:RESC1005X40N, F.Cu at (-43.7, 95.2)
- added R23: 22K, SamacSys_Parts:RESC1005X40N, F.Cu at (-43.7, 90.8)
- added R24: 12K 1%, Resistor_SMD:R_0402_1005Metric, F.Cu at (-35.8, 90.8)
- added R25: 470R, SamacSys_Parts:RESC1005X40N, F.Cu at (-20.8, 80.8)
- added R26: 1k, SamacSys_Parts:RESC1005X37N, F.Cu at (-20.8, 83.8)
- added R27: 12K 1%, Resistor_SMD:R_0402_1005Metric, F.Cu at (-66.5, 91.0)
- added R28: 470R, SamacSys_Parts:RESC1005X40N, F.Cu at (-51.0, 80.8)
- added R29: 1k, SamacSys_Parts:RESC1005X37N, F.Cu at (-51.0, 83.8)
- added R30: 100K, SamacSys_Parts:RESC1005X40N, F.Cu at (-49.5, 80.8)
- added R31: 22K, SamacSys_Parts:RESC1005X40N, F.Cu at (-49.5, 83.8)
- added R32: 100R, SamacSys_Parts:RESC1005X40N, F.Cu at (-47.5, 84.8)
- added R33: 1k, SamacSys_Parts:RESC1005X37N, F.Cu at (-44.0, 84.8)
- added R34: 100K, SamacSys_Parts:RESC1005X40N, F.Cu at (-19.2, 80.8)
- added R35: 22K, SamacSys_Parts:RESC1005X40N, F.Cu at (-19.2, 83.8)
- added R36: 100R, SamacSys_Parts:RESC1005X40N, F.Cu at (-17.5, 84.8)
- added R37: 1k, SamacSys_Parts:RESC1005X37N, F.Cu at (-13.8, 84.8)
- added R38: NF, SamacSys_Parts:RESC1005X40N, F.Cu at (-15.6, 135.9)
- added R39: 22K, SamacSys_Parts:RESC1005X40N, F.Cu at (-15.6, 138.1)
- added R4: NF, SamacSys_Parts:RESC1005X40N, F.Cu at (-43.7, 92.2)
- added R40: 22K, SamacSys_Parts:RESC1005X40N, F.Cu at (-15.6, 140.2)
- added R41: NF, SamacSys_Parts:RESC1005X40N, F.Cu at (-15.6, 142.4)
- added U3: STUSB4500QTR, Package_DFN_QFN:QFN-24-1EP_4x4mm_P0.5mm_EP2.7x2.7mm, F.Cu at (-28.3, 88.5)
- added U7: STUSB4500QTR, Package_DFN_QFN:QFN-24-1EP_4x4mm_P0.5mm_EP2.7x2.7mm, F.Cu at (-58.8, 88.8)
- moved J8 44.1 mm to (171.4, 127.7)
Connections:
- J2 pad 16: /Board_Edge_Connector/GPIO25 -> unconnected-(J2-Pad16)
- J2 pad 28: /Board_Edge_Connector/GPIO19 -> unconnected-(J2-Pad28)
- J2 pad 36: /Board_Edge_Connector/GPIO15 -> unconnected-(J2-Pad36)
- J8 pad 5: /Board_Edge_Connector/GPIO15 -> GND
Routing:
- net unconnected-(J2-Pad16): track 0.00 -> 89.6 mm, vias 0 -> 2
- net /Board_Edge_Connector/GPIO25: track 88.2 -> 0.00 mm, vias 2 -> 0
- net unconnected-(J2-Pad28): track 0.00 -> 87.8 mm, vias 0 -> 2
- net /Board_Edge_Connector/GPIO19: track 87.8 -> 0.00 mm, vias 2 -> 0
- net unconnected-(J2-Pad36): track 0.00 -> 85.3 mm, vias 0 -> 2
- net /Board_Edge_Connector/GPIO15: track 85.3 -> 0.00 mm, vias 2 -> 0
- net /Board_Edge_Connector/GPIO6: track 11.4 -> 92.1 mm, vias 0 -> 3
- net /Board_Edge_Connector/GPIO8: track 3.58 -> 82.8 mm, vias 1 -> 3
- net /Board_Edge_Connector/GPIO10: track 4.64 -> 81.5 mm, vias 0 -> 1
- net /Board_Edge_Connector/GPIO4: track 10.7 -> 77.8 mm, vias 0 -> 1
- net /Board_Edge_Connector/GPIO2: track 10.2 -> 75.5 mm, vias 0 -> 1
- net Net-(D18-CATHODE_1): track 0.00 -> 44.9 mm, vias 0 -> 2
- net GND: track 134.0 -> 176.1 mm, vias 77 -> 99
- net Net-(U7-DISCH): track 0.00 -> 21.4 mm, vias 0 -> 2
- net Net-(U7-VREG_1V2): track 0.00 -> 19.9 mm, vias 0 -> 2
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
Commit message: PWR regs complete, EMI protection? LDO low noise passthrough??
Parts:
- removed MOSFET1, MOSFET2: STL11N3LLH6, STL11N3LLH6:POWERFLAT_3P3X3P3_STM
- added C44: 1u, RESC2012X140N:RESC2012X140N, F.Cu at (37.0, 92.2)
- added C45: 1u, RESC2012X140N:RESC2012X140N, F.Cu at (37.0, 95.2)
- added C46: 1u, RESC2012X140N:RESC2012X140N, F.Cu at (37.0, 98.3)
- added C47: 100n, Capacitor_SMD:C_0402_1005Metric, F.Cu at (224.5, 69.0)
- added C48: 100n, Capacitor_SMD:C_0402_1005Metric, F.Cu at (233.2, 68.0)
- added C49: 10u, Capacitor_SMD:C_0805_2012Metric, F.Cu at (222.1, 62.5)
- added C50: 10u, Capacitor_SMD:C_0805_2012Metric, F.Cu at (222.1, 59.8)
- added IC4: LM74610QDGKRQ1, SamacSys_Parts:SOP65P490X110-8N, F.Cu at (43.0, 93.0)
- added IC5: LMR51450FNDRRR, SamacSys_Parts:SON50P300X300X80-13N-D, F.Cu at (229.0, 65.8)
- added J13: 1190297, SamacSys_Parts:1190297, F.Cu at (24.6, 78.0)
- added J3: PJ-102BH, SamacSys_Parts:PJ-102AH, F.Cu at (37.2, 84.9)
- added L1: IHLP2525EZER2R2M01-2.2uH, SamacSys_Parts:INDPM6965X500N, F.Cu at (229.0, 59.8)
- added Q3: STL11N3LLH6, STL11N3LLH6:POWERFLAT_3P3X3P3_STM, F.Cu at (176.5, 102.8)
- added Q4: STL11N3LLH6, STL11N3LLH6:POWERFLAT_3P3X3P3_STM, F.Cu at (184.7, 102.8)
- added Q5: STL11N3LLH6, STL11N3LLH6:POWERFLAT_3P3X3P3_STM, F.Cu at (23.1, 97.1)
- added R1: 100K, SamacSys_Parts:RESC1005X40N, F.Cu at (224.2, 64.5)
- added R3: 19K1, SamacSys_Parts:RESC1005X40N, F.Cu at (224.2, 66.0)
- added R42: 100K, SamacSys_Parts:RESC1005X40N, F.Cu at (233.0, 64.8)
- added R43: 13K3, SamacSys_Parts:RESC1005X40N, F.Cu at (224.2, 67.5)
- moved J12 253.5 mm to (188.2, 52.0), turned to 90 degrees
- moved D17 250.1 mm to (180.1, 48.7), turned to 90 degrees
- moved D16 247.6 mm to (177.1, 48.7), turned to 90 degrees
- moved R27 244.8 mm to (174.7, 49.5), turned to -90 degrees
- moved C36 242.1 mm to (184.5, 59.4), turned to 180 degrees
- moved U7 239.4 mm to (178.5, 56.5), turned to 180 degrees
- moved D18 238.8 mm to (184.4, 62.4), turned to 180 degrees
- moved R28 236.4 mm to (184.9, 65.0), turned to 180 degrees
- moved C37 236.0 mm to (181.0, 62.1), turned to 90 degrees
- moved R30 234.8 mm to (184.9, 66.5), turned to 180 degrees
- moved R29 233.7 mm to (181.9, 65.0), turned to 180 degrees
- moved R31 232.1 mm to (181.9, 66.5), turned to 180 degrees
- moved C34 230.9 mm to (176.0, 61.3), turned to 180 degrees
- moved Q2 230.7 mm to (184.5, 70.0), turned to -90 degrees
- moved R32 229.0 mm to (180.9, 68.5), turned to 180 degrees
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Connections:
- Module1 pad 26: /Board_Edge_Connector/GPIO19 -> GND
- Module1 pad 41: /Board_Edge_Connector/GPIO25 -> GND
- Module1 pad 51: /Board_Edge_Connector/GPIO15 -> GND
Routing:
- net GND: track 176.1 -> 221.7 mm, vias 99 -> 118
- net /Power_Input/USBC_PWR.Sheet/V_SINK: track 5.36 -> 50.1 mm
- net Net-(D14-CATHODE_1): track 10.5 -> 39.5 mm, vias 0 -> 2
- net Net-(U3-DISCH): track 0.00 -> 23.7 mm, vias 0 -> 2
- net /Power_Input/USBC_PWR.Sheet1/V_SINK: track 5.71 -> 28.5 mm
- net /Power_Input/USBC_PWR.Sheet1/ADDR1: track 0.00 -> 20.7 mm, vias 0 -> 3
- net /Power_Input/USBC_PWR.Sheet1/CC1: track 0.00 -> 19.1 mm, vias 0 -> 3
- net /Power_Input/USBC_PWR.Sheet1/ADDR0: track 0.00 -> 18.7 mm, vias 0 -> 2
- net +5V: track 12.5 -> 30.6 mm
- net Net-(IC5-SW_1): track 0.00 -> 15.0 mm
- net Net-(U3-VBUS_EN_SNK): track 0.00 -> 14.8 mm, vias 0 -> 2
- net +20V: track 0.00 -> 13.0 mm, vias 0 -> 25
- net Net-(U7-VREG_1V2): track 19.9 -> 7.26 mm
- net Net-(U3-VBUS_VS_DISCH): track 0.00 -> 11.7 mm, vias 0 -> 2
- net Net-(IC3-GATE_DRIVE): track 0.00 -> 11.1 mm
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- added copper zone on F.Cu, net +20V
