File: hardware/rpi-cm4-base-carrier/cm4-gpio.kicad_sch (KiCad schematic)
At the start: 1 part

Commit message: design files exported ready for manufacture, LCSC part numbers added throughout the library
Parts:
- Module1: LCSC Part # (none) -> C597931; LCSC Part Number (none) -> C597931
Other:
- title: Raspberry Pi Compute Module 4 Base Carrier -> Raspberry Pi Compute Module 4 Control Node
Changed lines of the file:
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@@
   (paper "A4")
   (title_block
-    (title "Raspberry Pi Compute Module 4 Base Carrier")
-    (date "2020-10-31")
+    (title "Raspberry Pi Compute Module 4 Control Node")
+    (date "2024-02-04")
     (rev "v01")
-    (comment 2 "creativecommons.org/licenses/by-sa/4.0")
+    (comment 2 "creativecommons.org/licenses/by-sa/4.0/")
     (comment 3 "License: CC BY-SA 4.0")
-    (comment 4 "Author: Shawn Hymel")
+    (comment 4 "Author: Sam Earnshaw")
   )
   (junction (at 54.61 62.23) (diameter 1.016) (color 0 0 0 0)
@@
       (effects (font (size 1.27 1.27)) hide)
     )
+    (property "LCSC Part Number" "C597931" (at 90.17 102.87 0)
+      (effects (font (size 1.27 1.27)) hide)
+    )
+    (property "LCSC Part #" "C597931" (at 90.17 102.87 0)
+      (effects (font (size 1.27 1.27)) hide)
+    )
