File: hardware/rpi-cm4-base-carrier/usbc_pwr.kicad_sch (KiCad schematic)
At the start: 19 parts, among them J3 USB4105-GF-A, Q2 STL6P3LLH6, U10 STUSB4500QTR

Commit message: design files exported ready for manufacture, LCSC part numbers added throughout the library
Parts:
- C1: LCSC Part # (none) -> C152724; LCSC Part Number (none) -> C152724
- C33, C34, C35, C37: LCSC Part # (none) -> C1849853; LCSC Part Number (none) -> C1849853
- C4: LCSC Part # (none) -> C326595; LCSC Part Number (none) -> C326595
- D15, D16, D17: LCSC Part # (none) -> C2935152; LCSC Part Number (none) -> C2935152
- J3: LCSC Part # (none) -> C2982555; LCSC Part Number (none) -> C2982555
- Q2: LCSC Part # (none) -> Non Stock; LCSC Part Number (none) -> Non Stock
- R24: LCSC Part # (none) -> C186129; LCSC Part Number (none) -> C186129
- R25, R29: LCSC Part # (none) -> C139047; LCSC Part Number (none) -> C139047
- R26: LCSC Part # (none) -> C131362; LCSC Part Number (none) -> C131362
- R27: LCSC Part # (none) -> C2576480; LCSC Part Number (none) -> C2576480
- R28: LCSC Part # (none) -> C186302; LCSC Part Number (none) -> C186302
- R9: LCSC Part # (none) -> C186350; LCSC Part Number (none) -> C186350
- U10: LCSC Part # (none) -> C2678061; LCSC Part Number (none) -> C2678061
Other:
- title: (none) -> Raspberry Pi Compute Module 4 Control Node
Changed lines of the file:
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@@
 (kicad_sch (version 20230121) (generator eeschema)
   (paper "A4")
+  (title_block
+    (title "Raspberry Pi Compute Module 4 Control Node")
+    (date "2024-02-04")
+    (comment 2 "creativecommons.org/licenses/by-sa/4.0/")
+    (comment 3 "License: CC BY-SA 4.0")
+    (comment 4 "Author: Sam Earnshaw")
+  )
   (junction (at 173.99 33.02) (diameter 0) (color 0 0 0 0)
   )
@@
       (effects (font (size 1.27 1.27)) (justify left top) hide)
     )
+    (property "LCSC Part Number" "C1849853" (at 44.45 99.06 0)
+      (effects (font (size 1.27 1.27)) hide)
+    )
+    (property "LCSC Part #" "C1849853" (at 44.45 99.06 0)
+      (effects (font (size 1.27 1.27)) hide)
+    )
     (pin "2")
     (pin "1")
@@
       (effects (font (size 1.27 1.27)) (justify left top) hide)
     )
+    (property "LCSC Part Number" "C2935152" (at 78.74 30.48 0)
+      (effects (font (size 1.27 1.27)) hide)
+    )
+    (property "LCSC Part #" "C2935152" (at 78.74 30.48 0)
+      (effects (font (size 1.27 1.27)) hide)
+    )
     (pin "2")
     (pin "3")
@@
       (effects (font (size 1.27 1.27)) (justify left top) hide)
     )
+    (property "LCSC Part Number" "C2935152" (at 43.18 123.19 0)
+      (effects (font (size 1.27 1.27)) hide)
+    )
+    (property "LCSC Part #" "C2935152" (at 43.18 123.19 0)
+      (effects (font (size 1.27 1.27)) hide)
+    )
     (pin "2")
     (pin "3")
@@
       (effects (font (size 1.27 1.27)) hide)
     )
+    (property "LCSC Part Number" "C186350" (at 58.42 107.95 0)
+      (effects (font (size 1.27 1.27)) hide)
+    )
+    (property "LCSC Part #" "C186350" (at 58.42 107.95 0)
+      (effects (font (size 1.27 1.27)) hide)
+    )
     (pin "1")
     (pin "2")
@@
     (property "Manufacturer_Part_Number" "08055C105JAT2A" (at -706.02 67.31 0)
       (effects (font (size 1.27 1.27)) (justify left top) hide)
+    )
+    (property "LCSC Part Number" "C1849853" (at 90.17 58.42 0)
+      (effects (font (size 1.27 1.27)) hide)
+    )
+    (property "LCSC Part #" "C1849853" (at 90.17 58.42 0)
+      (effects (font (size 1.27 1.27)) hide)
     )
     (pin "2")
@@
     (property "STANDARD" "Manufacturer Recommendations" (at 130.81 27.94 0)
       (effects (font (size 1.27 1.27)) (justify bottom) hide)
+    )
+    (property "LCSC Part Number" "Non Stock" (at 130.81 27.94 0)
+      (effects (font (size 1.27 1.27)) hide)
+    )
+    (property "LCSC Part #" "Non Stock" (at 130.81 27.94 0)
+      (effects (font (size 1.27 1.27)) hide)
     )
     (pin "2")
@@
       (effects (font (size 1.27 1.27)) (justify left top) hide)
     )
+    (property "LCSC Part Number" "C2935152" (at 24.13 123.19 0)
+      (effects (font (size 1.27 1.27)) hide)
+    )
+    (property "LCSC Part #" "C2935152" (at 24.13 123.19 0)
+      (effects (font (size 1.27 1.27)) hide)
+    )
     (pin "2")
     (pin "3")
@@
       (effects (font (size 1.27 1.27)) (justify left top) hide)
     )
+    (property "LCSC Part Number" "C1849853" (at 34.29 99.06 0)
+      (effects (font (size 1.27 1.27)) hide)
+    )
+    (property "LCSC Part #" "C1849853" (at 34.29 99.06 0)
+      (effects (font (size 1.27 1.27)) hide)
+    )
     (pin "2")
     (pin "1")
@@
       (effects (font (size 1.27 1.27)) (justify left top) hide)
     )
+    (property "LCSC Part Number" "C2576480" (at 119.38 53.34 0)
+      (effects (font (size 1.27 1.27)) hide)
+    )
+    (property "LCSC Part #" "C2576480" (at 119.38 53.34 0)
+      (effects (font (size 1.27 1.27)) hide)
+    )
     (pin "1")
     (pin "2")
@@
       (effects (font (size 1.27 1.27)) (justify left top) hide)
     )
+    (property "LCSC Part Number" "C131362" (at 119.38 30.48 0)
+      (effects (font (size 1.27 1.27)) hide)
+    )
+    (property "LCSC Part #" "C131362" (at 119.38 30.48 0)
+      (effects (font (size 1.27 1.27)) hide)
+    )
     (pin "2")
     (pin "1")
@@
       (effects (font (size 1.27 1.27)) hide)
     )
+    (property "LCSC Part Number" "C326595" (at 66.04 40.64 0)
+      (effects (font (size 1.27 1.27)) hide)
+    )
+    (property "LCSC Part #" "C326595" (at 66.04 40.64 0)
+      (effects (font (size 1.27 1.27)) hide)
+    )
     (pin "1")
     (pin "2")
@@
       (effects (font (size 1.27 1.27)) (justify left top) hide)
     )
+    (property "LCSC Part Number" "C139047" (at 100.33 53.34 0)
+      (effects (font (size 1.27 1.27)) hide)
+    )
+    (property "LCSC Part #" "C139047" (at 100.33 53.34 0)
+      (effects (font (size 1.27 1.27)) hide)
+    )
     (pin "2")
     (pin "1")
@@
     (property "Manufacturer_Part_Number" "CR0402-JW-471GLF" (at -695.86 44.45 0)
       (effects (font (size 1.27 1.27)) (justify left top) hide)
+    )
+    (property "LCSC Part Number" "C186129" (at 100.33 30.48 0)
+      (effects (font (size 1.27 1.27)) hide)
+    )
+    (property "LCSC Part #" "C186129" (at 100.33 30.48 0)
+      (effects (font (size 1.27 1.27)) hide)
     )
     (pin "2")
@@
     )
     (property "Digi-Key_PN" "2073-USB4105-GF-ACT-ND" (at 38.1 38.1 0)
+      (effects (font (size 1.27 1.27)) hide)
+    )
+    (property "LCSC Part Number" "C2982555" (at 38.1 38.1 0)
+      (effects (font (size 1.27 1.27)) hide)
+    )
+    (property "LCSC Part #" "C2982555" (at 38.1 38.1 0)
       (effects (font (size 1.27 1.27)) hide)
     )
@@
       (effects (font (size 1.27 1.27)) hide)
     )
+    (property "LCSC Part Number" "C152724" (at 189.23 38.1 0)
+      (effects (font (size 1.27 1.27)) hide)
+    )
+    (property "LCSC Part #" "C152724" (at 189.23 38.1 0)
+      (effects (font (size 1.27 1.27)) hide)
+    )
     (pin "1")
     (pin "2")
@@
       (effects (font (size 1.27 1.27)) (justify left top) hide)
     )
+    (property "LCSC Part Number" "C139047" (at 199.39 30.48 0)
+      (effects (font (size 1.27 1.27)) hide)
+    )
+    (property "LCSC Part #" "C139047" (at 199.39 30.48 0)
+      (effects (font (size 1.27 1.27)) hide)
+    )
     (pin "2")
     (pin "1")
@@
       (effects (font (size 1.27 1.27)) (justify left top) hide)
     )
+    (property "LCSC Part Number" "C1849853" (at 24.13 99.06 0)
+      (effects (font (size 1.27 1.27)) hide)
+    )
+    (property "LCSC Part #" "C1849853" (at 24.13 99.06 0)
+      (effects (font (size 1.27 1.27)) hide)
+    )
     (pin "2")
     (pin "1")
@@
     )
     (property "Datasheet" "https://www.st.com/resource/en/datasheet/stusb4500.pdf" (at 90.17 125.73 0)
+      (effects (font (size 1.27 1.27)) hide)
+    )
+    (property "LCSC Part Number" "C2678061" (at 90.17 125.73 0)
+      (effects (font (size 1.27 1.27)) hide)
+    )
+    (property "LCSC Part #" "C2678061" (at 90.17 125.73 0)
       (effects (font (size 1.27 1.27)) hide)
     )
@@
       (effects (font (size 1.27 1.27)) (justify left top) hide)
     )
+    (property "LCSC Part Number" "C186302" (at 168.91 50.8 0)
+      (effects (font (size 1.27 1.27)) hide)
+    )
+    (property "LCSC Part #" "C186302" (at 168.91 50.8 0)
+      (effects (font (size 1.27 1.27)) hide)
+    )
     (pin "2")
